Commit message: Fixed basic model
Basic model more accurate to base frame of the robot now.

File: ora_description/description/anteater_core.xacro (robot description, xacro)
@@ -24,5 +24,5 @@
   <link name="chassis_link">
     <visual>
-      <origin xyz="${base_length / 2} 0 ${base_height / 2}" rpy="0 0 0"/>
+      <origin xyz="${0 + (back_caster_x_offset / 4)} 0 ${back_caster_radius / 4}" rpy="0 0 0"/>
       <geometry>
         <box size="${base_length} ${base_width} ${base_height}"/>
@@ -31,5 +31,5 @@
     </visual>
     <collision>
-      <origin xyz="${base_length / 2} 0 ${base_height / 2}" rpy="0 0 0"/>
+      <origin xyz="${0 + (back_caster_x_offset / 4)} 0 ${back_caster_radius / 4}" rpy="0 0 0"/>
       <geometry>
         <box size="${base_length} ${base_width} ${base_height}"/>
@@ -37,5 +37,5 @@
     </collision>
     <xacro:inertial_box mass="10.0" x="${base_length}" y="${base_width}" z="${base_height}">
-      <origin xyz="${base_length / 2} 0 ${base_height / 2}" rpy="0 0 0"/>
+      <origin xyz="0 0 0" rpy="0 0 0"/>
     </xacro:inertial_box>
   </link>

File: ora_description/description/caster.xacro (robot description, xacro)
@@ -1,4 +1,6 @@
 <?xml version="1.0"?>
 <robot xmlns:xacro="http://www.ros.org/wiki/xacro" >
+  <xacro:include filename="dimensions.xacro"/>
+  <xacro:include filename="inertia_macros.xacro"/>
   <!--###############-->
   <!-- Front Casters -->
@@ -25,5 +27,5 @@
       <parent link="base_link"/>
       <child link="${prefix}_front_caster_link"/>
-      <origin xyz="${x_reflect*front_caster_x_offset} ${y_reflect*front_caster_y_offset} ${main_wheel_z_offset - front_caster_z_offset}" rpy="0 0 0"/>
+      <origin xyz="${x_reflect*front_caster_x_offset} ${y_reflect*front_caster_y_offset} ${-main_wheel_radius + front_caster_radius}" rpy="0 0 0"/>
       <axis xyz="0 1 0"/>
     </joint>
@@ -60,5 +62,5 @@
       <parent link="base_link"/>
       <child link="${prefix}_back_caster_link"/>
-      <origin xyz="${x_reflect*back_caster_x_offset} ${y_reflect*back_caster_y_offset} ${main_wheel_z_offset - back_caster_z_offset}" rpy="0 0 0"/>
+      <origin xyz="${x_reflect*back_caster_x_offset} ${y_reflect*back_caster_y_offset} ${-main_wheel_radius + back_caster_radius}" rpy="0 0 0"/>
       <axis xyz="0 1 0"/>
     </joint>

File: ora_description/description/dimensions.xacro (robot description, xacro)
@@ -9,7 +9,7 @@
   <xacro:property name="in_to_m" value="${0.0254}"/>
   <!-- Base Chassis Dimensions -->
-  <xacro:property name="base_length" value="${0.508}"/>
-  <xacro:property name="base_width" value="${0.406}"/>
-  <xacro:property name="base_height" value="${0.406}"/>
+  <xacro:property name="base_length" value="${34 * in_to_m}"/>
+  <xacro:property name="base_width" value="${17.5 * in_to_m}"/>
+  <xacro:property name="base_height" value="${10 * in_to_m}"/>
   <!-- Wheel Dimensions / Location -->
   <xacro:property name="main_wheel_diameter" value="${33.02 * cm_to_m}"/>

File: ora_description/description/wheel.xacro (robot description, xacro)
@@ -1,9 +1,11 @@
 <?xml version="1.0"?>
 <robot xmlns:xacro="http://www.ros.org/wiki/xacro" >
+  <xacro:include filename="dimensions.xacro"/>
+  <xacro:include filename="inertia_macros.xacro"/>
   <xacro:macro name="wheel" params="prefix x_reflect y_reflect">
     <joint name="${prefix}_wheel_joint" type="continuous">
       <parent link="base_link"/>
       <child link="${prefix}_wheel_link"/>
-      <origin xyz="${main_wheel_x_offset} ${main_wheel_y_offset} ${main_wheel_z_offset}" rpy="-${pi / 2} 0.0 0.0"/>
+      <origin xyz="${x_reflect * main_wheel_x_offset} ${y_reflect * main_wheel_y_offset} ${main_wheel_z_offset}" rpy="-${pi / 2} 0.0 0.0"/>
       <axis xyz="0 0 -1"/>
     </joint>
@@ -29,4 +31,4 @@
   </xacro:macro>
   <xacro:wheel prefix="left" x_reflect="1" y_reflect="1" />
-  <xacro:wheel prefix="right" x_reflect="1" y_reflect="-1" />
+  <xacro:wheel prefix="right" x_reflect="-1" y_reflect="-1" />
 </robot>

Commit message: Corrected errors in joints and Gazebo accel

File: ora_description/description/anteater_core.xacro (robot description, xacro)
@@ -36,5 +36,5 @@
       </geometry>
     </collision>
-    <xacro:inertial_box mass="10.0" x="${base_length}" y="${base_width}" z="${base_height}">
+    <xacro:inertial_box mass="50.0" x="${base_length}" y="${base_width}" z="${base_height}">
       <origin xyz="0 0 0" rpy="0 0 0"/>
     </xacro:inertial_box>

File: ora_description/description/caster.xacro (robot description, xacro)
@@ -30,5 +30,5 @@
       <axis xyz="0 1 0"/>
     </joint>
-    <gazebo reference="{prefix}_front_caster_link">
+    <gazebo reference="${prefix}_front_caster_link">
       <material>Gazebo/Black</material>
       <!-- Frictionless-ish -->
@@ -65,5 +65,5 @@
       <axis xyz="0 1 0"/>
     </joint>
-    <gazebo reference="{prefix}_back_caster_link">
+    <gazebo reference="${prefix}_back_caster_link">
       <material>Gazebo/Black</material>
       <!-- Frictionless-ish -->

File: ora_description/description/sensors.xacro (robot description, xacro)
@@ -95,8 +95,8 @@
       <right_joint>right_wheel_joint</right_joint>
       <!-- kinematics -->
-      <wheel_separation>0.4</wheel_separation>
+      <wheel_separation>${base_width}</wheel_separation>
       <wheel_radius>${main_wheel_radius}</wheel_radius>
       <!-- limits -->
-      <max_linear_acceleration>0.1</max_linear_acceleration>
+      <max_linear_acceleration>2.0</max_linear_acceleration>
       <!-- input -->
       <topic>/demo/cmd_vel</topic>

File: ora_description/description/wheel.xacro (robot description, xacro)
@@ -7,5 +7,5 @@
       <parent link="base_link"/>
       <child link="${prefix}_wheel_link"/>
-      <origin xyz="${x_reflect * main_wheel_x_offset} ${y_reflect * main_wheel_y_offset} ${main_wheel_z_offset}" rpy="-${pi / 2} 0.0 0.0"/>
+      <origin xyz="${x_reflect * main_wheel_x_offset} ${y_reflect * main_wheel_y_offset} ${main_wheel_z_offset}" rpy="${pi / 2} 0.0 0.0"/>
       <axis xyz="0 0 -1"/>
     </joint>

Commit message: Added sim LiDAR
Does not work yet, need to adjust

File: ora_description/description/anteater_core.xacro (robot description, xacro)
@@ -24,5 +24,5 @@
   <link name="chassis_link">
     <visual>
-      <origin xyz="${0 + (back_caster_x_offset / 4)} 0 ${back_caster_radius / 4}" rpy="0 0 0"/>
+      <origin xyz="${base_x_offset} 0 ${base_z_offset}" rpy="0 0 0"/>
       <geometry>
         <box size="${base_length} ${base_width} ${base_height}"/>

File: ora_description/description/dimensions.xacro (robot description, xacro)
@@ -32,3 +32,11 @@
   <xacro:property name="back_caster_y_offset" value="${26.9875 * cm_to_m}"/>
   <xacro:property name="back_caster_x_offset" value="${33.02 * cm_to_m}"/>
+  <!-- Lidar Dimensions -->
+  <xacro:property name="lidar_height" value="${71.7 * mm_to_m}"/>
+  <xacro:property name="lidar_radius" value="${103.3 * mm_to_m / 2}"/>
+  <!-- Assorted Offset Values -->
+  <xacro:property name="base_x_offset" value="${(back_caster_x_offset / 4)}"/>
+  <xacro:property name="base_z_offset" value="${back_caster_radius / 4}"/>
+  <xacro:property name="lidar_x_offset" value="${(base_length / 2) - (lidar_radius / 2) + (base_x_offset / 2)}"/>
+  <xacro:property name="lidar_z_offset" value="${(base_height / 2) + (lidar_height / 2) + base_z_offset}"/>
 </robot>

File: ora_description/description/sensors.xacro (robot description, xacro)
@@ -3,91 +3,149 @@
   <xacro:include filename="dimensions.xacro"/>
   <xacro:include filename="inertia_macros.xacro"/>
-  <gazebo>
-    <joint name='imu_joint' type='fixed'>
-      <parent>base_link</parent>
-      <child>imu_link</child>
-      <pose relative_to="base_link">0.0 0.0 0.01 0 0 0</pose>
-    </joint>
-    <link name='imu_link'>
-      <pose relative_to="imu_joint"/>
-      <visual name="imu_link_visual">
-          <geometry>
-            <box><size>
-                0.1 0.1 0.1
-            </size></box>
-          </geometry>
-      </visual>
-      <collision name="imu_link_collision">
-        <geometry>
-          <box><size>
-              0.1 0.1 0.1
-          </size></box>
-        </geometry>
-      </collision>
-      <xacro:inertial_box mass="0.1" x="0.1" y="0.1" z="0.1">
-        <origin xyz="0 0 0" rpy="0 0 0"/>
-      </xacro:inertial_box>
-      <sensor name="imu_sensor" type="imu">
-        <always_on>true</always_on>
-        <update_rate>100</update_rate>
-        <visualize>true</visualize>
-        <topic>demo/imu</topic>
-        <gz_frame_id>imu_link</gz_frame_id>
-        <imu>
-          <angular_velocity>
-            <x>
-              <noise type="gaussian">
+  <!-- Lidar -->
+  <link name="lidar_link">
+    <inertial>
+      <origin xyz="0 0 0" rpy="0 0 0"/>
+      <mass value="0.125"/>
+      <inertia ixx="0.001" ixy="0" ixz="0" iyy="0.001" iyz="0" izz="0.001" />
+    </inertial>
+    <collision>
+      <origin xyz="0 0 0" rpy="0 0 0"/>
+      <geometry>
+        <cylinder radius="${lidar_radius}" length="${lidar_height}"/>
+      </geometry>
+    </collision>
+    <visual>
+      <origin xyz="0 0 0" rpy="0 0 0"/>
+      <geometry>
+        <cylinder radius="${lidar_radius}" length="${lidar_height}"/>
+      </geometry>
+    </visual>
+  </link>
+  <joint name="lidar_joint" type="fixed">
+    <parent link="base_link"/>
+    <child link="lidar_link"/>
+    <origin xyz="${lidar_x_offset} 0 ${lidar_z_offset}" rpy="0 0 0"/>
+  </joint>
+  <!-- Lidar Plugin -->
+  <gazebo reference="lidar_link">
+    <sensor name="lidar" type="gpu_lidar">
+      <always_on>true</always_on>
+      <visualize>true</visualize>
+      <update_rate>5</update_rate>
+      <topic>scan</topic>
+      <gz_frame_id>lidar_link</gz_frame_id>
+      <lidar>
+        <scan>
+          <horizontal>
+            <samples>360</samples>
+            <resolution>1.000000</resolution>
+            <min_angle>0.000000</min_angle>
+            <max_angle>6.280000</max_angle>
+          </horizontal>
+        </scan>
+        <range>
+          <min>0.120000</min>
+          <max>3.5</max>
+          <resolution>0.015000</resolution>
+        </range>
+        <noise>
+          <type>gaussian</type>
+          <mean>0.0</mean>
+          <stddev>0.01</stddev>
+        </noise>
+      </lidar>
+    </sensor>
+  </gazebo>
+  <!-- IMU -->
+  <link name="imu_link">
+    <inertial>
+      <origin xyz="0 0 0" rpy="0 0 0"/>
+      <mass value="0.1"/>
+      <inertia ixx="0.0001" ixy="0" ixz="0" iyy="0.0001" iyz="0" izz="0.0001"/>
+    </inertial>
+    <visual>
+      <origin xyz="0 0 0" rpy="0 0 0"/>
+      <geometry>
+        <box size="0.1 0.1 0.1"/>
+      </geometry>
+    </visual>
+    <collision>
+      <origin xyz="0 0 0" rpy="0 0 0"/>
+      <geometry>
+        <box size="0.1 0.1 0.1"/>
+      </geometry>
+    </collision>
+  </link>
+  <joint name="imu_joint" type="fixed">
+    <parent link="base_link"/>
+    <child link="imu_link"/>
+    <origin xyz="0 0 0.01" rpy="0 0 0"/>
+  </joint>
+  <!-- IMU Plugin -->
+  <gazebo reference="imu_link">
+    <sensor name="imu_sensor" type="imu">
+      <always_on>true</always_on>
+      <update_rate>100</update_rate>
+      <visualize>true</visualize>
+      <topic>demo/imu</topic>
+      <gz_frame_id>imu_link</gz_frame_id>
+      <imu>
+        <angular_velocity>
+          <x>
+            <noise type="gaussian">
+              <mean>0.0</mean>
+              <stddev>2e-4</stddev>
+              <bias_mean>0.0000075</bias_mean>
+              <bias_stddev>0.0000008</bias_stddev>
+            </noise>
+          </x>
+          <y>
+            <noise type="gaussian">
+              <mean>0.0</mean>
+              <stddev>2e-4</stddev>
+              <bias_mean>0.0000075</bias_mean>
+              <bias_stddev>0.0000008</bias_stddev>
+            </noise>
+          </y>
+          <z>
+            <noise type="gaussian">
                 <mean>0.0</mean>
                 <stddev>2e-4</stddev>
                 <bias_mean>0.0000075</bias_mean>
                 <bias_stddev>0.0000008</bias_stddev>
-              </noise>
-            </x>
-            <y>
-              <noise type="gaussian">
+            </noise>
+          </z>
+        </angular_velocity>
+      <linear_acceleration>
+          <x>
+            <noise type="gaussian">
                 <mean>0.0</mean>
-                <stddev>2e-4</stddev>
-                <bias_mean>0.0000075</bias_mean>
-                <bias_stddev>0.0000008</bias_stddev>
-              </noise>
-            </y>
-            <z>
-              <noise type="gaussian">
-                  <mean>0.0</mean>
-                  <stddev>2e-4</stddev>
-                  <bias_mean>0.0000075</bias_mean>
-                  <bias_stddev>0.0000008</bias_stddev>
-              </noise>
-            </z>
-          </angular_velocity>
-        <linear_acceleration>
-            <x>
-              <noise type="gaussian">
-                  <mean>0.0</mean>
-                  <stddev>1.7e-2</stddev>
-                  <bias_mean>0.1</bias_mean>
-                  <bias_stddev>0.001</bias_stddev>
-              </noise>
-            </x>
-            <y>
-              <noise type="gaussian">
-                  <mean>0.0</mean>
-                  <stddev>1.7e-2</stddev>
-                  <bias_mean>0.1</bias_mean>
-                  <bias_stddev>0.001</bias_stddev>
-              </noise>
-            </y>
-            <z>
-              <noise type="gaussian">
-                  <mean>0.0</mean>
-                  <stddev>1.7e-2</stddev>
-                  <bias_mean>0.1</bias_mean>
-                  <bias_stddev>0.001</bias_stddev>
-              </noise>
-            </z>
-          </linear_acceleration>
-        </imu>
-      </sensor>
-    </link>
+                <stddev>1.7e-2</stddev>
+                <bias_mean>0.1</bias_mean>
+                <bias_stddev>0.001</bias_stddev>
+            </noise>
+          </x>
+          <y>
+            <noise type="gaussian">
+                <mean>0.0</mean>
+                <stddev>1.7e-2</stddev>
+                <bias_mean>0.1</bias_mean>
+                <bias_stddev>0.001</bias_stddev>
+            </noise>
+          </y>
+          <z>
+            <noise type="gaussian">
+                <mean>0.0</mean>
+                <stddev>1.7e-2</stddev>
+                <bias_mean>0.1</bias_mean>
+                <bias_stddev>0.001</bias_stddev>
+            </noise>
+          </z>
+        </linear_acceleration>
+      </imu>
+    </sensor>
+  </gazebo>
+  <gazebo>
     <plugin filename="gz-sim-diff-drive-system" name="gz::sim::systems::DiffDrive">
       <!-- wheels -->
