Commit message: Fixed issues with spawning robot in gazebo
Robot moves weirdly, gotta fix that

File: ora_description/description/anteater.urdf.xacro (robot description, xacro)
@@ -8,3 +8,4 @@
   <xacro:include filename="caster.xacro"/>
   <xacro:include filename="wheel.xacro"/>
+  <xacro:include filename="sensors.xacro"/>
 </robot>

File: ora_description/description/sensors.xacro (robot description, xacro)
@@ -1,12 +1,22 @@
 <?xml version="1.0"?>
 <robot xmlns:xacro="https://www.ros.org/wiki/xacro">
-  <joint name='imu_joint' type='fixed'>
-    <parent>base_link</parent>
-    <child>imu_link</child>
-    <pose relative_to="base_link">0.0 0.0 0.01 0 0 0</pose>
-  </joint>
-  <link name='imu_link'>
-    <pose relative_to="imu_joint"/>
-    <visual name="imu_link_visual">
+  <xacro:include filename="dimensions.xacro"/>
+  <xacro:include filename="inertia_macros.xacro"/>
+  <gazebo>
+    <joint name='imu_joint' type='fixed'>
+      <parent>base_link</parent>
+      <child>imu_link</child>
+      <pose relative_to="base_link">0.0 0.0 0.01 0 0 0</pose>
+    </joint>
+    <link name='imu_link'>
+      <pose relative_to="imu_joint"/>
+      <visual name="imu_link_visual">
+          <geometry>
+            <box><size>
+                0.1 0.1 0.1
+            </size></box>
+          </geometry>
+      </visual>
+      <collision name="imu_link_collision">
         <geometry>
           <box><size>
@@ -14,96 +24,92 @@
           </size></box>
         </geometry>
-    </visual>
-    <collision name="imu_link_collision">
-      <geometry>
-        <box><size>
-            0.1 0.1 0.1
-        </size></box>
-      </geometry>
-    </collision>
-    <xacro:box_inertia m="0.1" w="0.1" d="0.1" h="0.1"/>
-    <sensor name="imu_sensor" type="imu">
-      <always_on>true</always_on>
-      <update_rate>100</update_rate>
-      <visualize>true</visualize>
-      <topic>demo/imu</topic>
-      <gz_frame_id>imu_link</gz_frame_id>
-      <imu>
-        <angular_velocity>
-          <x>
-            <noise type="gaussian">
-              <mean>0.0</mean>
-              <stddev>2e-4</stddev>
-              <bias_mean>0.0000075</bias_mean>
-              <bias_stddev>0.0000008</bias_stddev>
-            </noise>
-          </x>
-          <y>
-            <noise type="gaussian">
-              <mean>0.0</mean>
-              <stddev>2e-4</stddev>
-              <bias_mean>0.0000075</bias_mean>
-              <bias_stddev>0.0000008</bias_stddev>
-            </noise>
-          </y>
-          <z>
-            <noise type="gaussian">
+      </collision>
+      <xacro:inertial_box mass="0.1" x="0.1" y="0.1" z="0.1">
+        <origin xyz="0 0 0" rpy="0 0 0"/>
+      </xacro:inertial_box>
+      <sensor name="imu_sensor" type="imu">
+        <always_on>true</always_on>
+        <update_rate>100</update_rate>
+        <visualize>true</visualize>
+        <topic>demo/imu</topic>
+        <gz_frame_id>imu_link</gz_frame_id>
+        <imu>
+          <angular_velocity>
+            <x>
+              <noise type="gaussian">
                 <mean>0.0</mean>
                 <stddev>2e-4</stddev>
                 <bias_mean>0.0000075</bias_mean>
                 <bias_stddev>0.0000008</bias_stddev>
-            </noise>
-          </z>
-        </angular_velocity>
-      <linear_acceleration>
-          <x>
-            <noise type="gaussian">
+              </noise>
+            </x>
+            <y>
+              <noise type="gaussian">
                 <mean>0.0</mean>
-                <stddev>1.7e-2</stddev>
-                <bias_mean>0.1</bias_mean>
-                <bias_stddev>0.001</bias_stddev>
-            </noise>
-          </x>
-          <y>
-            <noise type="gaussian">
-                <mean>0.0</mean>
-                <stddev>1.7e-2</stddev>
-                <bias_mean>0.1</bias_mean>
-                <bias_stddev>0.001</bias_stddev>
-            </noise>
-          </y>
-          <z>
-            <noise type="gaussian">
-                <mean>0.0</mean>
-                <stddev>1.7e-2</stddev>
-                <bias_mean>0.1</bias_mean>
-                <bias_stddev>0.001</bias_stddev>
-            </noise>
-          </z>
-        </linear_acceleration>
-      </imu>
-    </sensor>
-  </link>
-  <plugin filename="gz-sim-diff-drive-system" name="gz::sim::systems::DiffDrive">
-    <!-- wheels -->
-    <left_joint>left_wheel_joint</left_joint>
-    <right_joint>right_wheel_joint</right_joint>
-    <!-- kinematics -->
-    <wheel_separation>0.4</wheel_separation>
-    <wheel_radius>${wheel_radius}</wheel_radius>
-    <!-- limits -->
-    <max_linear_acceleration>0.1</max_linear_acceleration>
-    <!-- input -->
-    <topic>/demo/cmd_vel</topic>
-    <!-- output -->
-    <odom_topic>/demo/odom</odom_topic>
-    <tf_topic>/tf</tf_topic>
-    <frame_id>odom</frame_id>
-    <child_frame_id>base_link</child_frame_id>
-  </plugin>
-  <plugin
-    filename="gz-sim-joint-state-publisher-system"
-    name="gz::sim::systems::JointStatePublisher">
-    <topic>joint_states</topic>
-  </plugin>
+                <stddev>2e-4</stddev>
+                <bias_mean>0.0000075</bias_mean>
+                <bias_stddev>0.0000008</bias_stddev>
+              </noise>
+            </y>
+            <z>
+              <noise type="gaussian">
+                  <mean>0.0</mean>
+                  <stddev>2e-4</stddev>
+                  <bias_mean>0.0000075</bias_mean>
+                  <bias_stddev>0.0000008</bias_stddev>
+              </noise>
+            </z>
+          </angular_velocity>
+        <linear_acceleration>
+            <x>
+              <noise type="gaussian">
+                  <mean>0.0</mean>
+                  <stddev>1.7e-2</stddev>
+                  <bias_mean>0.1</bias_mean>
+                  <bias_stddev>0.001</bias_stddev>
+              </noise>
+            </x>
+            <y>
+              <noise type="gaussian">
+                  <mean>0.0</mean>
+                  <stddev>1.7e-2</stddev>
+                  <bias_mean>0.1</bias_mean>
+                  <bias_stddev>0.001</bias_stddev>
+              </noise>
+            </y>
+            <z>
+              <noise type="gaussian">
+                  <mean>0.0</mean>
+                  <stddev>1.7e-2</stddev>
+                  <bias_mean>0.1</bias_mean>
+                  <bias_stddev>0.001</bias_stddev>
+              </noise>
+            </z>
+          </linear_acceleration>
+        </imu>
+      </sensor>
+    </link>
+    <plugin filename="gz-sim-diff-drive-system" name="gz::sim::systems::DiffDrive">
+      <!-- wheels -->
+      <left_joint>left_wheel_joint</left_joint>
+      <right_joint>right_wheel_joint</right_joint>
+      <!-- kinematics -->
+      <wheel_separation>0.4</wheel_separation>
+      <wheel_radius>${main_wheel_radius}</wheel_radius>
+      <!-- limits -->
+      <max_linear_acceleration>0.1</max_linear_acceleration>
+      <!-- input -->
+      <topic>/demo/cmd_vel</topic>
+      <!-- output -->
+      <odom_topic>/demo/odom</odom_topic>
+      <tf_topic>/tf</tf_topic>
+      <frame_id>odom</frame_id>
+      <child_frame_id>base_link</child_frame_id>
+    </plugin>
+    <plugin
+      filename="gz-sim-joint-state-publisher-system"
+      name="gz::sim::systems::JointStatePublisher">
+      <topic>joint_states</topic>
+    </plugin>
+  </gazebo>
 </robot>

File: ora_description/description/wheel.xacro (robot description, xacro)
@@ -30,5 +30,5 @@
     </gazebo>
   </xacro:macro>
-  <xacro:wheel prefix="left" x_reflect="1" y_reflect="1" />
-  <xacro:wheel prefix="right" x_reflect="-1" y_reflect="-1" />
+  <xacro:wheel prefix="left" x_reflect="-1" y_reflect="1" />
+  <xacro:wheel prefix="right" x_reflect="1" y_reflect="-1" />
 </robot>

Commit message: Added real robot ros2_control

File: ora_description/description/anteater.urdf.xacro (robot description, xacro)
@@ -1,4 +1,5 @@
 <?xml version="1.0"?>
 <robot xmlns:xacro="https://www.ros.org/wiki/xacro" name="robot_name">
+  <xacro:arg name="sim_mode" default="false"/>
   <!-- Include all of the pieces of the robot -->
   <xacro:include filename="anteater_core.xacro"/>

File: ora_description/description/ros2_control.xacro (robot description, xacro)
@@ -1,6 +1,4 @@
 <?xml version="1.0"?>
 <robot xmlns:xacro="https://www.ros.org/wiki/xacro">
-  <!-- Args -->
-  <xacro:arg name="sim_mode" default="true"/>
   <xacro:if value="$(arg sim_mode)">
     <ros2_control name="GazeboSystem" type="system">
@@ -52,5 +50,24 @@
   </xacro:if>
   <xacro:unless value="$(arg sim_mode)">
-    <!-- TODO: Add real hardware control -->
+    <ros2_control name="RealRobot" type="system">
+      <hardware>
+        <plugin>roboteq_ros2_control_plugin/RoboteqHardwareInterface</plugin>
+        <param name="can">can0</param>
+      </hardware>
+      <joint name="left_wheel_joint">
+        <param name="node_id">1</param>
+        <param name="gear_ratio">7.3</param>
+        <command_interface name="velocity"/>
+        <state_interface name="velocity"/>
+        <state_interface name="position"/>
+      </joint>
+      <joint name="right_wheel_joint">
+        <param name="node_id">2</param>
+        <param name="gear_ratio">7.3</param>
+        <command_interface name="velocity"/>
+        <state_interface name="velocity"/>
+        <state_interface name="position"/>
+      </joint>
+    </ros2_control>
   </xacro:unless>
 </robot>
